File: cdfr2024-pamis/cdfr2024-pamis.kicad_pcb (KiCad board)
At the start: 4 copper layers, 75.7 x 64.3 mm, 24 parts, among them J1 Connecteur batterie, J2 Conn_ST_STDC14, J3 Connecteur Programmation, J4 Connecteur Débug, J5 Connecteur ToF, J6 Moteur Droit, J7 Moteur Gauche, U1 STM32F401RCTx, U2 LM317_SOT-223, U4 Driver Moteur Droit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

Commit message: module wifi
Parts:
- removed C2, C3, C4, C5: 100nF, Capacitor_SMD:C_0805_2012Metric_Pad1.18x1.45mm_HandSolder
- removed C6: 4.7uF, Capacitor_SMD:C_0805_2012Metric_Pad1.18x1.45mm_HandSolder
- removed C7: 10nF, Capacitor_SMD:C_0805_2012Metric_Pad1.18x1.45mm_HandSolder
- removed C8: 1uF, Capacitor_SMD:C_0805_2012Metric_Pad1.18x1.45mm_HandSolder
- removed J2: Conn_ST_STDC14, FTSH-107-01-L-DV-K-A:SAMTEC_FTSH-107-01-L-DV-K-A
- removed J3: Connecteur Programmation, Connector_PinHeader_2.54mm:PinHeader_1x04_P2.54mm_Vertical
- removed J4: Connecteur Débug, Connector_PinHeader_2.54mm:PinHeader_1x03_P2.54mm_Vertical
- removed R4: 10k, Resistor_SMD:R_0805_2012Metric_Pad1.20x1.40mm_HandSolder
- removed U1: STM32F401RCTx, Package_QFP:LQFP-64_10x10mm_P0.5mm
- added U3: ESP32-S3-DEVKITC-1-N8R2, ESP32S3-devkit:ESP32-S3-DEVKITC, F.Cu at (85.1, 68.1)
- U4, U5: footprint A4988_Stepper_Motor_Driver:MODULE_A4988_STEPPER_MOTOR_DRIVER_CARRIER -> A4988:MODULE_A4988_STEPPER_MOTOR_DRIVER_CARRIER
- moved J6 78.7 mm to (48.3, 76.2)
- moved U2 62.4 mm to (118.7, 48.1), turned to 0 degrees
- moved U4 59.3 mm to (60.7, 80.9)
- moved R2 47.6 mm to (107.5, 43.0), turned to 180 degrees
- moved C1 47.5 mm to (111.1, 63.3), turned to 180 degrees
- moved R3 43.2 mm to (107.5, 48.1), turned to 180 degrees
- moved J5 43.1 mm to (85.1, 78.2), turned to 180 degrees
- moved R1 37.7 mm to (107.5, 37.9), turned to 180 degrees
- moved J1 30.8 mm to (119.5, 75.2)
- moved D1 30.6 mm to (107.5, 53.1)
- moved J7 28.1 mm to (49.1, 55.8), turned to 180 degrees
- moved U5 5.88 mm to (60.4, 52.5), turned to 180 degrees
Routing:
- net +3.3V: track 301.2 -> 0.00 mm, vias 5 -> 0
- net GND: track 223.4 -> 0.00 mm, vias 7 -> 0
- net +7.5V: track 162.9 -> 0.00 mm
- net SWDIO: track 83.1 -> 0.00 mm, vias 1 -> 0
- net /RX: track 73.8 -> 0.00 mm, vias 2 -> 0
- net Net-(U2-ADJ): track 70.9 -> 0.00 mm
- net /TX: track 61.2 -> 0.00 mm, vias 2 -> 0
- net RST: track 56.9 -> 0.00 mm, vias 2 -> 0
- net Net-(U3-GPIO2): track 56.0 -> 0.00 mm, vias 1 -> 0
- net SWCLK: track 47.5 -> 0.00 mm
- net Net-(U1-BOOT0): track 45.8 -> 0.00 mm, vias 2 -> 0
- net Net-(U3-GPIO3): track 42.5 -> 0.00 mm
- net Net-(U3-GPIO0): track 41.9 -> 0.00 mm, vias 1 -> 0
- net Net-(U1-VCAP1): track 40.9 -> 0.00 mm, vias 2 -> 0
- net Net-(U3-GPIO4): track 40.7 -> 0.00 mm
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- removed copper zone on In1.Cu, net GND

Commit message: Routage + DRC
Parts:
- added J3: Connecteur RF, Connector_PinHeader_2.54mm:PinHeader_1x04_P2.54mm_Vertical, F.Cu at (115.8, 103.9)
- moved J5 32.1 mm to (77.7, 109.5), turned to 90 degrees
- moved U4 7.13 mm to (65.3, 75.4), turned to 180 degrees
- moved J6 6.52 mm to (54.1, 79.2), turned to 180 degrees
- moved J7 5.49 mm to (54.4, 54.1)
- moved U5 4.88 mm to (64.8, 50.3)
- moved U3 3.97 mm to (87.6, 71.1)
- moved R1 0.81 mm to (107.5, 37.1), turned to 0 degrees
Connections:
- U3 pad J1_13: Net-(U3-GPIO3) -> unconnected-(U3-GPIO3-PadJ1_13)
- U3 pad J1_15: Net-(U3-GPIO9) -> unconnected-(U3-GPIO9-PadJ1_15)
- U3 pad J1_16: Net-(U3-GPIO10) -> unconnected-(U3-GPIO10-PadJ1_16)
- U3 pad J1_20: Net-(U3-GPIO14) -> unconnected-(U3-GPIO14-PadJ1_20)
- U3 pad J1_4: Net-(U3-GPIO4) -> unconnected-(U3-GPIO4-PadJ1_4)
- U3 pad J1_5: Net-(U3-GPIO5) -> unconnected-(U3-GPIO5-PadJ1_5)
- U3 pad J3_2: unconnected-(U3-U0TXD/GPIO43-PadJ3_2) -> Net-(J3-Pin_3)
- U3 pad J3_3: unconnected-(U3-U0RXD/GPIO44-PadJ3_3) -> Net-(J3-Pin_2)
- U4 pad 5: Net-(U3-GPIO11) -> unconnected-(U4-M2-Pad5)
- U4 pad 6: Net-(U3-GPIO12) -> unconnected-(U4-M1-Pad6)
- U4 pad 7: Net-(U3-GPIO13) -> unconnected-(U4-M0-Pad7)
- U5 pad 5: Net-(U3-GPIO2) -> unconnected-(U5-M2-Pad5)
- U5 pad 6: Net-(U3-GPIO3) -> unconnected-(U5-M1-Pad6)
- U5 pad 7: Net-(U3-GPIO4) -> unconnected-(U5-M0-Pad7)
- U5 pad 8: Net-(U3-GPIO5) -> Net-(U3-GPIO2)
Routing:
- net +7.5V: track 0.00 -> 147.7 mm, vias 0 -> 2
- net +3.3V: track 0.00 -> 112.0 mm
- net Net-(U3-GPIO0): track 0.00 -> 69.0 mm, vias 0 -> 1
- net Net-(J3-Pin_2): track 0.00 -> 62.8 mm
- net Net-(J3-Pin_3): track 0.00 -> 62.1 mm
- net Net-(J5-Pin_4): track 0.00 -> 53.8 mm
- net GND: track 0.00 -> 50.0 mm
- net Net-(J5-Pin_6): track 0.00 -> 49.0 mm
- net Net-(U3-GPIO1): track 0.00 -> 48.8 mm
- net Net-(J5-Pin_7): track 0.00 -> 45.9 mm
- net Net-(J5-Pin_2): track 0.00 -> 44.6 mm
- net Net-(J5-Pin_8): track 0.00 -> 43.3 mm
- net Net-(J5-Pin_3): track 0.00 -> 41.0 mm
- net Net-(J5-Pin_9): track 0.00 -> 40.4 mm
- net Net-(J5-Pin_5): track 0.00 -> 39.5 mm, vias 0 -> 2
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- added copper zone on In2.Cu, net +3.3V
- added copper zone on In1.Cu, net GND
Other:
- board size 75.7 x 64.3 mm -> 75.6 x 95.7 mm
