File: cdfr2024-pamis/cdfr2024-pamis.kicad_pcb (KiCad board)
At the start: 4 copper layers, 75.6 x 95.7 mm, 14 parts, among them J1 Connecteur batterie, J3 Connecteur RF, J5 Connecteur ToF, J6 Moteur Droit, J7 Moteur Gauche, U2 LM317_SOT-223, U3 ESP32-S3-DEVKITC-1-N8R2, U4 Driver Moteur Droit, U5 Driver Moteur Gauche

Commit message: carte fablab module rf
Parts:
- removed J3: Connecteur RF, Connector_PinHeader_2.54mm:PinHeader_1x04_P2.54mm_Vertical
- removed J6: Moteur Droit, Connector_PinHeader_2.54mm:PinHeader_1x04_P2.54mm_Vertical
- removed U3: ESP32-S3-DEVKITC-1-N8R2, ESP32S3-devkit:ESP32-S3-DEVKITC
- added J2: Connecteur Bouton, Connector_PinHeader_2.54mm:PinHeader_1x02_P2.54mm_Vertical, F.Cu at (70.6, 49.4)
- added J4: Moteur Droit, Connector_PinHeader_2.54mm:PinHeader_1x04_P2.54mm_Vertical, F.Cu at (124.8, 62.9)
- added J8: Connecteur RF, Connector_PinHeader_2.54mm:PinHeader_1x08_P2.54mm_Vertical, F.Cu at (98.8, 122.0)
- added U1: ESP32-DEVKIT-V1, ESP32DevkitV1:MODULE_ESP32_DEVKIT_V1, F.Cu at (89.2, 87.8)
- moved J1 67.9 mm to (63.0, 37.6)
- moved J5 50.3 mm to (119.8, 81.9), turned to 0 degrees
- moved U4 48.9 mm to (113.4, 66.9), turned to 0 degrees
- moved C1 38.2 mm to (80.2, 40.8)
- moved U5 31.4 mm to (63.3, 81.6)
- moved J7 31.0 mm to (52.8, 85.1)
- moved R3 18.6 mm to (93.9, 35.5)
- moved D1 18.1 mm to (103.7, 35.4)
- moved R1 15.6 mm to (93.9, 44.8)
- moved U2 15.4 mm to (103.3, 48.3)
- moved R2 13.9 mm to (93.9, 39.9)
Connections:
- C1 pad 1: +3.3V -> +3V3
- D1 pad 2: +3.3V -> +3V3
- J1 pad 1: +7.5V -> Net-(J1-Pin_1)
- J5 pad 2: Net-(J5-Pin_2) -> +3V3
- J5 pad 3: Net-(J5-Pin_3) -> +3V3
- J5 pad 6: Net-(J5-Pin_6) -> /SCL
- J5 pad 7: Net-(J5-Pin_7) -> /SDA
- R1 pad 1: +3.3V -> +3V3
- U2 pad 2: +3.3V -> +3V3
- U4 pad 10: +3.3V -> +3V3
- U5 pad 10: +3.3V -> +3V3
Routing:
- net +3V3: track 0.00 -> 318.4 mm, vias 0 -> 9
- net GND: track 50.0 -> 310.0 mm, vias 0 -> 5
- net +3.3V: track 112.0 -> 0.00 mm
- net /SDA: track 0.00 -> 88.0 mm, vias 0 -> 2
- net /SCL: track 0.00 -> 77.6 mm, vias 0 -> 2
- net Net-(J3-Pin_2): track 62.8 -> 0.00 mm
- net Net-(J3-Pin_3): track 62.1 -> 0.00 mm
- net Net-(U1-D5): track 69.0 -> 7.02 mm, vias 1 -> 0
- net /SCLK: track 0.00 -> 54.0 mm
- net Net-(J5-Pin_6): track 49.0 -> 0.00 mm
- net +7.5V: track 147.7 -> 100.6 mm
- net Net-(J5-Pin_7): track 45.9 -> 0.00 mm
- net Net-(J5-Pin_2): track 44.6 -> 0.00 mm
- net Net-(J5-Pin_3): track 41.0 -> 0.00 mm
- net Net-(J8-Pin_1): track 0.00 -> 39.6 mm
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- added copper zone on In2.Cu, net +3V3
- removed copper zone on In2.Cu, net +3.3V
