File: cdfr2024-pamis/cdfr2024-pamis.kicad_pcb (KiCad board)
At the start: 4 copper layers, 75.6 x 95.7 mm, 15 parts, among them J1 Connecteur batterie, J2 Connecteur Bouton, J4 Moteur Droit, J5 Connecteur ToF, J7 Moteur Gauche, J8 Connecteur RF, U1 ESP32-DEVKIT-V1, U2 LM317_SOT-223, U4 Driver Moteur Droit, U5 Driver Moteur Gauche

Commit message: carte pamis
Parts:
- removed C1: 100uF, Capacitor_SMD:CP_Elec_10x10.5
- removed D1: LED, LED_SMD:LED_0805_2012Metric_Pad1.15x1.40mm_HandSolder
- removed J8: Connecteur RF, Connector_PinHeader_2.54mm:PinHeader_1x08_P2.54mm_Vertical
- removed R1: 2k4, Resistor_SMD:R_0805_2012Metric_Pad1.20x1.40mm_HandSolder
- removed R2: 3k9, Resistor_SMD:R_0805_2012Metric_Pad1.20x1.40mm_HandSolder
- removed R3: 150, Resistor_SMD:R_0805_2012Metric_Pad1.20x1.40mm_HandSolder
- removed U2: LM317_SOT-223, Package_TO_SOT_SMD:SOT-223-3_TabPin2
- added J3: Connecteur RF, Connector_PinHeader_2.54mm:PinHeader_1x12_P2.54mm_Vertical, F.Cu at (82.7, 54.2)
- added J6: Module MP1584EN, MP1584EN_Module:SRT_MPT1584EN_Module, F.Cu at (81.2, 41.1)
- moved J4 73.1 mm to (67.9, 108.8), turned to -90 degrees
- moved U4 57.8 mm to (64.1, 97.2), turned to -90 degrees
- moved J5 51.7 mm to (98.2, 34.9)
- moved J7 46.0 mm to (92.3, 108.6), turned to -90 degrees
- moved U5 29.6 mm to (88.5, 97.2), turned to -90 degrees
- moved U1 20.0 mm to (76.6, 72.3), turned to -90 degrees
- moved J2 10.4 mm to (67.4, 39.5)
- moved J1 8.65 mm to (56.3, 43.0), turned to 0 degrees
Connections:
- net /SCL renamed /EVK_SCL
- net /SDA renamed /EVK_SDA
- net Net-(J5-Pin_4) renamed /EVK_EN
- J5 pad 5: Net-(J5-Pin_5) -> /EVK_LPN
- J5 pad 8: Net-(J5-Pin_8) -> /EVK_RST
- J5 pad 9: Net-(J5-Pin_9) -> /EVK_INT
- U1 pad 10: /SDI -> /RF_SDI
- U1 pad 15: /SDO -> /RF_SDO
- U1 pad 16: +3V3 -> unconnected-(U1-EN-Pad16)
- U1 pad 19: Net-(J8-Pin_3) -> unconnected-(U1-D34-Pad19)
- U1 pad 20: Net-(J8-Pin_2) -> unconnected-(U1-D35-Pad20)
- U1 pad 21: Net-(J8-Pin_1) -> /DR_STEPD
- U1 pad 22: Net-(J5-Pin_9) -> /DR_DIRD
- U1 pad 23: Net-(J5-Pin_8) -> /DR_STEPG
- U1 pad 24: Net-(J5-Pin_5) -> /DR_DIRG
- U1 pad 26: Net-(U1-D14) -> /EVK_LPN
- U1 pad 27: Net-(U1-D12) -> /EVK_RST
- U1 pad 28: Net-(U1-D13) -> /EVK_INT
- U1 pad 30: +3V3 -> unconnected-(U1-VIN-Pad30)
- U1 pad 4: Net-(U1-D2) -> /RF_2
- U1 pad 5: Net-(U1-D4) -> /RF_3
- U1 pad 8: Net-(U1-D5) -> /RF_4
- U1 pad 9: /SCLK -> /RF_SCLK
- U4 pad 1: Net-(U1-D14) -> /DR_DIRD
- U4 pad 2: Net-(U1-D13) -> /DR_STEPD
- U4 pad 3: unconnected-(U4-Pad3) -> Net-(U4-Pad3)
- U4 pad 4: unconnected-(U4-Pad4) -> Net-(U4-Pad3)
- U4 pad 8: Net-(U1-D12) -> unconnected-(U4-~{ENABLE}-Pad8)
- U5 pad 1: Net-(U1-D5) -> /DR_DIRG
- U5 pad 2: Net-(U1-D4) -> /DR_STEPG
- U5 pad 3: unconnected-(U5-Pad3) -> Net-(U5-Pad3)
- U5 pad 4: unconnected-(U5-Pad4) -> Net-(U5-Pad3)
- U5 pad 8: Net-(U1-D2) -> unconnected-(U5-~{ENABLE}-Pad8)
Routing:
- net +3V3: track 318.4 -> 164.6 mm, vias 9 -> 6
- net /SCLK: track 54.0 -> 0.00 mm
- net /EVK_LPN: track 0.00 -> 50.5 mm, vias 0 -> 2
- net /EVK_RST: track 0.00 -> 43.3 mm
- net /EVK_SDA: track 88.0 -> 46.0 mm, vias 2 -> 0
- net Net-(J8-Pin_1): track 39.6 -> 0.00 mm
- net /EVK_INT: track 0.00 -> 37.8 mm
- net Net-(U1-D14): track 37.4 -> 0.00 mm
- net /EVK_EN: track 19.8 -> 57.1 mm, vias 0 -> 2
- net +7.5V: track 100.6 -> 137.6 mm, vias 2 -> 3
- net Net-(J8-Pin_2): track 36.1 -> 0.00 mm
- net /SDI: track 34.0 -> 0.00 mm
- net GND: track 310.0 -> 279.8 mm, vias 5 -> 6
- net /RF_SDO: track 0.00 -> 29.7 mm
- net /SDO: track 26.8 -> 0.00 mm
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- added copper zone on In1.Cu, net +3V3
- removed copper zone on In1.Cu, net GND
Other:
- board size 75.6 x 95.7 mm -> 50 x 80 mm
